File: src/Downloader/LEDBlinker/Hardware/KiCad/LEDBlinker/LEDBlinker.kicad_pcb (KiCad board)
At the start: 2 copper layers, 68.6 x 33 mm, 4 parts, among them SW1 1825910-6, U1 Heltec_HTIT-WB32

Commit message: Updated silkscreen
Other:
- board text added: "LED Blinker for BatteryServer_V3 https://github.com/HBoyd255/BatteryServer_V3 Board: V1"
- board text removed: "LED Blinker for BatteryServer_V3 https://github.com/H-Boyd/BatteryServer_V3 Board: V1"
